File: pcb/I2C-Signal.sch (KiCad schematic (older format))
At the start: 11 parts, among them J13 SM04B-SRSS-TB(LF)(SN), J17 SM04B-SRSS-TB(LF)(SN), J7 Conn_01x04_Male, J8 Conn_01x04_Male, U6 PCA9306DCTR

Commit message: Changed some values - RC for the inputs to lower frequencys, reduced lines on the BOM by some minor value changes
Parts:
- C23: value 100p -> 1n
Changed lines of the file:
@@
 AR Path="/5CA10EE5/5CA193D5" Ref="C23"  Part="1"
 F 0 "C23" V 4148 2700 50  0000 C CNN
-F 1 "100p" V 4239 2700 50  0000 C CNN
+F 1 "1n" V 4239 2700 50  0000 C CNN
 F 2 "Capacitor_SMD:C_0805_2012Metric" H 4438 2550 50  0001 C CNN
 F 3 "~" H 4400 2700 50  0001 C CNN
