File: pcb/LAN8720.sch (KiCad schematic (older format))
At the start: 23 parts, among them J15 RJ45_Amphenol_RJMG1BD3B8K1ANR, U11 LAN8720A

Commit message: changed connection of the LAN8720A, RST to the FXL6408 and MDIO to the ESP32 (where RST was before). fixes #2
Connections:
- net MDIO: now reaches U11.12 (MDIO)
Changed lines of the file:
@@
 Text Label 2550 3750 0    50   ~ 0
 TD-
+Text HLabel 10050 3250 2    50   BiDi ~ 0
+MDIO
+Wire Wire Line
+	10050 3250 6100 3250
 $EndSCHEMATC
