File: pcb/ADS-Input.sch (KiCad schematic (older format))
At the start: 13 parts, among them J10 Conn_01x02_Male, J13 Conn_01x04_Male, U7 ADS1115IDGS, U8 PCA9306DCTR

Commit message: first version of the new feature set
Parts:
- removed C22: 100p, Capacitor_SMD:C_0805_2012Metric_Pad1.15x1.40mm_HandSolder, symbol Device:C
- removed J10: Conn_01x02_Male, Connector_PinHeader_2.54mm:PinHeader_1x02_P2.54mm_Vertical, symbol Connector:Conn_01x02_Male
- removed J13: Conn_01x04_Male, Connector_PinHeader_2.54mm:PinHeader_1x04_P2.54mm_Vertical, symbol Connector:Conn_01x04_Male
- removed R19: 220k, Resistor_SMD:R_0805_2012Metric_Pad1.15x1.40mm_HandSolder, symbol Device:R
- removed R20, R21: 2.4k, Resistor_SMD:R_0805_2012Metric_Pad1.15x1.40mm_HandSolder, symbol Device:R
- removed U8: PCA9306DCTR, Package_SO:SSOP-8_2.95x2.8mm_P0.65mm, symbol Interface:PCA9306
- added C16: 100p, Capacitor_SMD:C_0805_2012Metric, symbol Device:C
- added C20: 22u, Capacitor_SMD:C_0805_2012Metric, symbol Device:C
- added J5: PTSM-Header-Horizontal-5, Connector_own:1814870, symbol Connector_own:PTSM-Header-Horizontal-5
- added L1: 22u, Inductor_SMD:L_0805_2012Metric, symbol Device:L
- added R22: 2.4k, Resistor_SMD:R_0805_2012Metric, symbol Device:R
- added R25: 240, Resistor_SMD:R_0805_2012Metric, symbol Device:R
- C17: renamed from C19; footprint Capacitor_SMD:C_0805_2012Metric_Pad1.15x1.40mm_HandSolder -> Capacitor_SMD:C_0805_2012Metric
- C18: renamed from C20; footprint Capacitor_SMD:C_0805_2012Metric_Pad1.15x1.40mm_HandSolder -> Capacitor_SMD:C_0805_2012Metric
- C19: renamed from C21; footprint Capacitor_SMD:C_0805_2012Metric_Pad1.15x1.40mm_HandSolder -> Capacitor_SMD:C_0805_2012Metric
- R23: renamed from R17; footprint Resistor_SMD:R_0805_2012Metric_Pad1.15x1.40mm_HandSolder -> Resistor_SMD:R_0805_2012Metric
- R24: renamed from R18; footprint Resistor_SMD:R_0805_2012Metric_Pad1.15x1.40mm_HandSolder -> Resistor_SMD:R_0805_2012Metric
- renumbered U7 to U4
Connections:
- net 5V: now also L1.2; no longer C19.1, U4.6 (AIN2), U4.8 (VDD)
- net GND: now also C16.2, C20.2, J5.3; no longer U4.7 (AIN3)
- net SCL: now also U4.10 (SCL)
- net SDA: now also U4.9 (SDA)
- net IN_B: no longer names the net of R23.2
- net IN_B: now also J5.2
- net In_A: no longer names the net of R24.2
- net In_A: now also J5.1
- new net: C19.1, C20.1, L1.1, R25.1, U4.8 (VDD)
- new net: C16.1, R22.1, U4.6 (AIN2)
- new net: J5.4, R25.2, U4.7 (AIN3)
- new net: J5.5, R22.2
Other:
- moved on the sheet: C17, C18, C19, R23, R24, U4

Commit message: Changed some values - RC for the inputs to lower frequencys, reduced lines on the BOM by some minor value changes
Parts:
- C16, C17, C18: value 100p -> 1n
- R22, R23, R24: value 2.4k -> 47k
- R25: value 240 -> 120
Changed lines of the file:
@@
 P 4150 3000
 F 0 "R24" V 3943 3000 50  0000 C CNN
-F 1 "2.4k" V 4034 3000 50  0000 C CNN
+F 1 "47k" V 4034 3000 50  0000 C CNN
 F 2 "Resistor_SMD:R_0805_2012Metric" V 4080 3000 50  0001 C CNN
 F 3 "~" H 4150 3000 50  0001 C CNN
@@
 P 3250 3200
 F 0 "R23" V 3043 3200 50  0000 C CNN
-F 1 "2.4k" V 3134 3200 50  0000 C CNN
+F 1 "47k" V 3134 3200 50  0000 C CNN
 F 2 "Resistor_SMD:R_0805_2012Metric" V 3180 3200 50  0001 C CNN
 F 3 "~" H 3250 3200 50  0001 C CNN
@@
 P 4400 3850
 F 0 "C17" H 4515 3896 50  0000 L CNN
-F 1 "100p" H 4515 3805 50  0000 L CNN
+F 1 "1n" H 4515 3805 50  0000 L CNN
 F 2 "Capacitor_SMD:C_0805_2012Metric" H 4438 3700 50  0001 C CNN
 F 3 "~" H 4400 3850 50  0001 C CNN
@@
 P 4900 3850
 F 0 "C18" H 5015 3896 50  0000 L CNN
-F 1 "100p" H 5015 3805 50  0000 L CNN
+F 1 "1n" H 5015 3805 50  0000 L CNN
 F 2 "Capacitor_SMD:C_0805_2012Metric" H 4938 3700 50  0001 C CNN
 F 3 "~" H 4900 3850 50  0001 C CNN
@@
 P 5400 2050
 F 0 "R25" V 5193 2050 50  0000 C CNN
-F 1 "240" V 5284 2050 50  0000 C CNN
+F 1 "120" V 5284 2050 50  0000 C CNN
 F 2 "Resistor_SMD:R_0805_2012Metric" V 5330 2050 50  0001 C CNN
 F 3 "~" H 5400 2050 50  0001 C CNN
@@
 P 3900 3850
 F 0 "C16" H 4015 3896 50  0000 L CNN
-F 1 "100p" H 4015 3805 50  0000 L CNN
+F 1 "1n" H 4015 3805 50  0000 L CNN
 F 2 "Capacitor_SMD:C_0805_2012Metric" H 3938 3700 50  0001 C CNN
 F 3 "~" H 3900 3850 50  0001 C CNN
@@
 P 2350 3400
 F 0 "R22" V 2143 3400 50  0000 C CNN
-F 1 "2.4k" V 2234 3400 50  0000 C CNN
+F 1 "47k" V 2234 3400 50  0000 C CNN
 F 2 "Resistor_SMD:R_0805_2012Metric" V 2280 3400 50  0001 C CNN
 F 3 "~" H 2350 3400 50  0001 C CNN

Commit message: Removed inductor in front of ADS1115, replaced with resistor (RC should be enough, comparison with the RC on the LSM9DS1 did not show many differences)
Parts:
- R2: renamed from L1; value 22u -> 24; footprint Inductor_SMD:L_0805_2012Metric -> Resistor_SMD:R_0805_2012Metric; symbol Device:L -> Device:R
Changed lines of the file:
@@
 Connection ~ 7550 2350
 $Comp
-L Device:L L1
+L Device:R R2
 U 1 1 5CA41C10
 P 8800 2050
-F 0 "L1" V 8990 2050 50  0000 C CNN
-F 1 "22u" V 8899 2050 50  0000 C CNN
-F 2 "Inductor_SMD:L_0805_2012Metric" H 8800 2050 50  0001 C CNN
+F 0 "R2" V 8990 2050 50  0000 C CNN
+F 1 "24" V 8899 2050 50  0000 C CNN
+F 2 "Resistor_SMD:R_0805_2012Metric" H 8800 2050 50  0001 C CNN
 F 3 "~" H 8800 2050 50  0001 C CNN
 	1    8800 2050
